File: MCU.kicad_sch (KiCad schematic)
At the start: 36 parts, among them J2 Conn_01x02_Pin, J3 Conn_01x02_Pin, J4 Conn_ARM_SWD_TagConnect_TC203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, U2 STM32H742VGH6, Y1 ABM3B-24.000MHZ

Commit message: Changed some of the silkscreen, and added some LEDs attached to some gpio
Parts:
- added D1, D2: Yellow, PCM_SparkFun-LED:LED_0603_1608Metric_Yellow, symbol PCM_SparkFun-LED:LED_Yellow_0603
- added D3, D4: Red, PCM_SparkFun-LED:LED_0603_1608Metric_Red, symbol PCM_SparkFun-LED:LED_Red_0603
- added R10, R11, R8, R9: R_Small_US, Resistor_SMD:R_0402_1005Metric, symbol Device:R_Small_US
Connections:
- net GND: now also R10.1, R11.1, R8.1, R9.1
- net PD14: now also D1.2 (A)
- net PD15: now also D2.2 (A)
- net PE14: now also D3.2 (A)
- net PE15: now also D4.2 (A)
- new net GPIO_LED1: D1.1 (K), R8.2
- new net GPIO_LED2: D2.1 (K), R9.2
- new net GPIO_LED3: D3.1 (K), R10.2
- new net GPIO_LED4: D4.1 (K), R11.2
Other:
- moved on the sheet: J4
