File: Memory.kicad_sch (KiCad schematic)
At the start: 12 parts, among them IC1 ${DEVICE}, J5 Micro_SD_Card_Det2, U3 W25Q128JVP

Commit message: Changed some of the silkscreen, and added some LEDs attached to some gpio
Parts:
- renumbered R8 to R12, R9 to R13, R10 to R14, R11 to R15, R12 to R16, R13 to R17
Changed lines of the file:
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@@
 		(in_pos_files yes)
 		(dnp no)
-		(property "Reference" "R12"
+		(property "Reference" "R16"
 			(at 219.71 107.9499 0)
 			(show_name no)
@@
 			(project "LSR_FLCM0001_A03"
 				(path "/1e96c69b-f36f-4762-8445-55c423e1825d/a1cb5f65-dcb2-46fb-a360-150ad6ab13b6"
-					(reference "R12")
+					(reference "R16")
 					(unit 1)
 					(variant
@@
 		(in_pos_files yes)
 		(dnp no)
-		(property "Reference" "R8"
+		(property "Reference" "R12"
 			(at 189.23 107.9499 0)
 			(show_name no)
@@
 			(project "LSR_FLCM0001_A03"
 				(path "/1e96c69b-f36f-4762-8445-55c423e1825d/a1cb5f65-dcb2-46fb-a360-150ad6ab13b6"
-					(reference "R8")
+					(reference "R12")
 					(unit 1)
 					(variant
@@
 		(in_pos_files yes)
 		(dnp no)
-		(property "Reference" "R11"
+		(property "Reference" "R15"
 			(at 212.09 107.9499 0)
 			(show_name no)
@@
 			(project "LSR_FLCM0001_A03"
 				(path "/1e96c69b-f36f-4762-8445-55c423e1825d/a1cb5f65-dcb2-46fb-a360-150ad6ab13b6"
-					(reference "R11")
+					(reference "R15")
 					(unit 1)
 					(variant
@@
 		(dnp no)
 		(fields_autoplaced yes)
-		(property "Reference" "#PWR039"
+		(property "Reference" "#PWR043"
 			(at 96.52 140.97 0)
 			(hide yes)
@@
 			(project "LSR_FLCM0001_A03"
 				(path "/1e96c69b-f36f-4762-8445-55c423e1825d/a1cb5f65-dcb2-46fb-a360-150ad6ab13b6"
-					(reference "#PWR039")
+					(reference "#PWR043")
 					(unit 1)
 				)
@@
 		(dnp no)
 		(fields_autoplaced yes)
-		(property "Reference" "#PWR045"
+		(property "Reference" "#PWR049"
 			(at 228.6 109.22 0)
 			(hide yes)
@@
 			(project "LSR_FLCM0001_A03"
 				(path "/1e96c69b-f36f-4762-8445-55c423e1825d/a1cb5f65-dcb2-46fb-a360-150ad6ab13b6"
-					(reference "#PWR045")
+					(reference "#PWR049")
 					(unit 1)
 				)
@@
 		(dnp no)
 		(fields_autoplaced yes)
-		(property "Reference" "#PWR042"
+		(property "Reference" "#PWR046"
 			(at 218.44 143.51 0)
 			(hide yes)
@@
 			(project "LSR_FLCM0001_A03"
 				(path "/1e96c69b-f36f-4762-8445-55c423e1825d/a1cb5f65-dcb2-46fb-a360-150ad6ab13b6"
-					(reference "#PWR042")
+					(reference "#PWR046")
 					(unit 1)
 				)
@@
 		(dnp no)
 		(fields_autoplaced yes)
-		(property "Reference" "#PWR043"
+		(property "Reference" "#PWR047"
 			(at 222.25 144.78 0)
 			(hide yes)
@@
 			(project "LSR_FLCM0001_A03"
 				(path "/1e96c69b-f36f-4762-8445-55c423e1825d/a1cb5f65-dcb2-46fb-a360-150ad6ab13b6"
-					(reference "#PWR043")
+					(reference "#PWR047")
 					(unit 1)
 				)
@@
 		(in_pos_files yes)
 		(dnp no)
-		(property "Reference" "R10"
+		(property "Reference" "R14"
 			(at 204.47 107.9499 0)
 			(show_name no)
@@
 			(project "LSR_FLCM0001_A03"
 				(path "/1e96c69b-f36f-4762-8445-55c423e1825d/a1cb5f65-dcb2-46fb-a360-150ad6ab13b6"
-					(reference "R10")
+					(reference "R14")
 					(unit 1)
 					(variant
@@
 		(in_pos_files yes)
 		(dnp no)
-		(property "Reference" "R13"
+		(property "Reference" "R17"
 			(at 220.98 143.5099 0)
 			(show_name no)
@@
 			(project "LSR_FLCM0001_A03"
 				(path "/1e96c69b-f36f-4762-8445-55c423e1825d/a1cb5f65-dcb2-46fb-a360-150ad6ab13b6"
-					(reference "R13")
+					(reference "R17")
 					(unit 1)
 					(variant
@@
 		(dnp no)
 		(fields_autoplaced yes)
-		(property "Reference" "#PWR036"
+		(property "Reference" "#PWR040"
 			(at 87.63 41.91 0)
 			(hide yes)
@@
 			(project "LSR_FLCM0001_A03"
 				(path "/1e96c69b-f36f-4762-8445-55c423e1825d/a1cb5f65-dcb2-46fb-a360-150ad6ab13b6"
-					(reference "#PWR036")
+					(reference "#PWR040")
 					(unit 1)
 				)
@@
 		(dnp no)
 		(fields_autoplaced yes)
-		(property "Reference" "#PWR046"
+		(property "Reference" "#PWR050"
 			(at 269.24 144.78 0)
 			(hide yes)
@@
 			(project "LSR_FLCM0001_A03"
 				(path "/1e96c69b-f36f-4762-8445-55c423e1825d/a1cb5f65-dcb2-46fb-a360-150ad6ab13b6"
-					(reference "#PWR046")
+					(reference "#PWR050")
 					(unit 1)
 				)
@@
 		(dnp no)
 		(fields_autoplaced yes)
-		(property "Reference" "#PWR033"
+		(property "Reference" "#PWR037"
 			(at 72.39 36.83 0)
 			(hide yes)
@@
 			(project "LSR_FLCM0001_A03"
 				(path "/1e96c69b-f36f-4762-8445-55c423e1825d/a1cb5f65-dcb2-46fb-a360-150ad6ab13b6"
-					(reference "#PWR033")
+					(reference "#PWR037")
 					(unit 1)
 				)
@@
 		(dnp no)
 		(fields_autoplaced yes)
-		(property "Reference" "#PWR044"
+		(property "Reference" "#PWR048"
 			(at 228.6 101.6 0)
 			(hide yes)
@@
 			(project "LSR_FLCM0001_A03"
 				(path "/1e96c69b-f36f-4762-8445-55c423e1825d/a1cb5f65-dcb2-46fb-a360-150ad6ab13b6"
-					(reference "#PWR044")
+					(reference "#PWR048")
 					(unit 1)
 				)
@@
 		(dnp no)
 		(fields_autoplaced yes)
-		(property "Reference" "#PWR040"
+		(property "Reference" "#PWR044"
 			(at 96.52 148.59 0)
 			(hide yes)
@@
 			(project "LSR_FLCM0001_A03"
 				(path "/1e96c69b-f36f-4762-8445-55c423e1825d/a1cb5f65-dcb2-46fb-a360-150ad6ab13b6"
-					(reference "#PWR040")
+					(reference "#PWR044")
 					(unit 1)
 				)
@@
 		(dnp no)
 		(fields_autoplaced yes)
-		(property "Reference" "#PWR037"
+		(property "Reference" "#PWR041"
 			(at 90.17 147.32 0)
 			(hide yes)
@@
 			(project "LSR_FLCM0001_A03"
 				(path "/1e96c69b-f36f-4762-8445-55c423e1825d/a1cb5f65-dcb2-46fb-a360-150ad6ab13b6"
-					(reference "#PWR037")
+					(reference "#PWR041")
 					(unit 1)
 				)
@@
 		(in_pos_files yes)
 		(dnp no)
-		(property "Reference" "R9"
+		(property "Reference" "R13"
 			(at 196.85 107.9499 0)
 			(show_name no)
@@
 			(project "LSR_FLCM0001_A03"
 				(path "/1e96c69b-f36f-4762-8445-55c423e1825d/a1cb5f65-dcb2-46fb-a360-150ad6ab13b6"
-					(reference "R9")
+					(reference "R13")
 					(unit 1)
 					(variant
@@
 		(dnp no)
 		(fields_autoplaced yes)
-		(property "Reference" "#PWR041"
+		(property "Reference" "#PWR045"
 			(at 186.69 107.95 0)
 			(hide yes)
@@
 			(project "LSR_FLCM0001_A03"
 				(path "/1e96c69b-f36f-4762-8445-55c423e1825d/a1cb5f65-dcb2-46fb-a360-150ad6ab13b6"
-					(reference "#PWR041")
+					(reference "#PWR045")
 					(unit 1)
 				)
@@
 		(dnp no)
 		(fields_autoplaced yes)
-		(property "Reference" "#PWR034"
+		(property "Reference" "#PWR038"
 			(at 72.39 64.77 0)
 			(hide yes)
@@
 			(project "LSR_FLCM0001_A03"
 				(path "/1e96c69b-f36f-4762-8445-55c423e1825d/a1cb5f65-dcb2-46fb-a360-150ad6ab13b6"
-					(reference "#PWR034")
+					(reference "#PWR038")
 					(unit 1)
 				)
@@
 		(dnp no)
 		(fields_autoplaced yes)
-		(property "Reference" "#PWR038"
+		(property "Reference" "#PWR042"
 			(at 90.17 154.94 0)
 			(hide yes)
@@
 			(project "LSR_FLCM0001_A03"
 				(path "/1e96c69b-f36f-4762-8445-55c423e1825d/a1cb5f65-dcb2-46fb-a360-150ad6ab13b6"
-					(reference "#PWR038")
+					(reference "#PWR042")
 					(unit 1)
 				)
@@
 		(dnp no)
 		(fields_autoplaced yes)
-		(property "Reference" "#PWR035"
+		(property "Reference" "#PWR039"
 			(at 87.63 34.29 0)
 			(hide yes)
@@
 			(project "LSR_FLCM0001_A03"
 				(path "/1e96c69b-f36f-4762-8445-55c423e1825d/a1cb5f65-dcb2-46fb-a360-150ad6ab13b6"
-					(reference "#PWR035")
+					(reference "#PWR039")
 					(unit 1)
 				)
