File: Power.kicad_sch (KiCad schematic)
At the start: 29 parts, among them J6 2125280200, U4 TPS62130A, U5 TPS2121RUXR

Commit message: Changed some of the silkscreen, and added some LEDs attached to some gpio
Parts:
- removed TP16: TestPoint, PCM_SparkFun-Connector:TestPoint-0.5mm, symbol Connector:TestPoint
- renumbered D1 to D5, D2 to D6, D3 to D7, D4 to D8, R14 to R18, R15 to R19, R16 to R20, R17 to R21, R18 to R22, R19 to R23, R20 to R24, R21 to R25, R22 to R26, R23 to R27, R24 to R28, TP17 to TP16, TP18 to TP17, TP19 to TP18
