File: Pyro.kicad_sch (KiCad schematic)
At the start: 19 parts, among them J7 1771114, Q1 AON7296, Q2 AON7296, Q3 AON7296

Commit message: Changed some of the silkscreen, and added some LEDs attached to some gpio
Parts:
- renumbered D6 to D10, D7 to D11, D5 to D9, R25 to R29, R26 to R30, R27 to R31, R28 to R32, R29 to R33, R30 to R34, R31 to R35, R32 to R36, R33 to R37, R34 to R38, R35 to R39, R36 to R40
Changed lines of the file:
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@@
 		(in_pos_files yes)
 		(dnp no)
-		(property "Reference" "R28"
+		(property "Reference" "R32"
 			(at 107.95 107.9499 0)
 			(show_name no)
@@
 			(project "LSR_FLCM0001_A03"
 				(path "/1e96c69b-f36f-4762-8445-55c423e1825d/3509533b-a3f9-46e2-8669-77eba5e31bfb"
-					(reference "R28")
+					(reference "R32")
 					(unit 1)
 					(variant
@@
 		(dnp no)
 		(fields_autoplaced yes)
-		(property "Reference" "#PWR079"
+		(property "Reference" "#PWR083"
 			(at 105.41 125.73 0)
 			(hide yes)
@@
 			(project "LSR_FLCM0001_A03"
 				(path "/1e96c69b-f36f-4762-8445-55c423e1825d/3509533b-a3f9-46e2-8669-77eba5e31bfb"
-					(reference "#PWR079")
+					(reference "#PWR083")
 					(unit 1)
 				)
@@
 		(in_pos_files yes)
 		(dnp no)
-		(property "Reference" "R30"
+		(property "Reference" "R34"
 			(at 107.95 149.8599 0)
 			(show_name no)
@@
 			(project "LSR_FLCM0001_A03"
 				(path "/1e96c69b-f36f-4762-8445-55c423e1825d/3509533b-a3f9-46e2-8669-77eba5e31bfb"
-					(reference "R30")
+					(reference "R34")
 					(unit 1)
 					(variant
@@
 		(in_pos_files yes)
 		(dnp no)
-		(property "Reference" "R31"
+		(property "Reference" "R35"
 			(at 107.95 157.4799 0)
 			(show_name no)
@@
 			(project "LSR_FLCM0001_A03"
 				(path "/1e96c69b-f36f-4762-8445-55c423e1825d/3509533b-a3f9-46e2-8669-77eba5e31bfb"
-					(reference "R31")
+					(reference "R35")
 					(unit 1)
 					(variant
@@
 		(in_pos_files yes)
 		(dnp no)
-		(property "Reference" "R29"
+		(property "Reference" "R33"
 			(at 107.95 115.5699 0)
 			(show_name no)
@@
 			(project "LSR_FLCM0001_A03"
 				(path "/1e96c69b-f36f-4762-8445-55c423e1825d/3509533b-a3f9-46e2-8669-77eba5e31bfb"
-					(reference "R29")
+					(reference "R33")
 					(unit 1)
 					(variant
@@
 		(in_pos_files yes)
 		(dnp no)
-		(property "Reference" "R36"
+		(property "Reference" "R40"
 			(at 116.84 68.5799 0)
 			(show_name no)
@@
 			(project "LSR_FLCM0001_A03"
 				(path "/1e96c69b-f36f-4762-8445-55c423e1825d/3509533b-a3f9-46e2-8669-77eba5e31bfb"
-					(reference "R36")
+					(reference "R40")
 					(unit 1)
 					(variant
@@
 		(dnp no)
 		(fields_autoplaced yes)
-		(property "Reference" "D7"
+		(property "Reference" "D11"
 			(at 116.84 60.8964 90)
 			(show_name no)
@@
 			(project "LSR_FLCM0001_A03"
 				(path "/1e96c69b-f36f-4762-8445-55c423e1825d/3509533b-a3f9-46e2-8669-77eba5e31bfb"
-					(reference "D7")
+					(reference "D11")
 					(unit 1)
 					(variant
@@
 		(dnp no)
 		(fields_autoplaced yes)
-		(property "Reference" "#PWR080"
+		(property "Reference" "#PWR084"
 			(at 105.41 167.64 0)
 			(hide yes)
@@
 			(project "LSR_FLCM0001_A03"
 				(path "/1e96c69b-f36f-4762-8445-55c423e1825d/3509533b-a3f9-46e2-8669-77eba5e31bfb"
-					(reference "#PWR080")
+					(reference "#PWR084")
 					(unit 1)
 				)
@@
 		(in_pos_files yes)
 		(dnp no)
-		(property "Reference" "R35"
+		(property "Reference" "R39"
 			(at 115.57 157.4799 0)
 			(show_name no)
@@
 			(project "LSR_FLCM0001_A03"
 				(path "/1e96c69b-f36f-4762-8445-55c423e1825d/3509533b-a3f9-46e2-8669-77eba5e31bfb"
-					(reference "R35")
+					(reference "R39")
 					(unit 1)
 					(variant
@@
 		(in_pos_files yes)
 		(dnp no)
-		(property "Reference" "R33"
+		(property "Reference" "R37"
 			(at 109.22 68.5799 0)
 			(show_name no)
@@
 			(project "LSR_FLCM0001_A03"
 				(path "/1e96c69b-f36f-4762-8445-55c423e1825d/3509533b-a3f9-46e2-8669-77eba5e31bfb"
-					(reference "R33")
+					(reference "R37")
 					(unit 1)
 					(variant
@@
 		(dnp no)
 		(fields_autoplaced yes)
-		(property "Reference" "#PWR082"
+		(property "Reference" "#PWR086"
 			(at 113.03 125.73 0)
 			(hide yes)
@@
 			(project "LSR_FLCM0001_A03"
 				(path "/1e96c69b-f36f-4762-8445-55c423e1825d/3509533b-a3f9-46e2-8669-77eba5e31bfb"
-					(reference "#PWR082")
+					(reference "#PWR086")
 					(unit 1)
 				)
@@
 		(dnp no)
 		(fields_autoplaced yes)
-		(property "Reference" "#PWR085"
+		(property "Reference" "#PWR089"
 			(at 167.64 55.88 0)
 			(hide yes)
@@
 			(project "LSR_FLCM0001_A03"
 				(path "/1e96c69b-f36f-4762-8445-55c423e1825d/3509533b-a3f9-46e2-8669-77eba5e31bfb"
-					(reference "#PWR085")
+					(reference "#PWR089")
 					(unit 1)
 				)
@@
 		(in_pos_files yes)
 		(dnp no)
-		(property "Reference" "R34"
+		(property "Reference" "R38"
 			(at 115.57 115.5699 0)
 			(show_name no)
@@
 			(project "LSR_FLCM0001_A03"
 				(path "/1e96c69b-f36f-4762-8445-55c423e1825d/3509533b-a3f9-46e2-8669-77eba5e31bfb"
-					(reference "R34")
+					(reference "R38")
 					(unit 1)
 					(variant
@@
 		(dnp no)
 		(fields_autoplaced yes)
-		(property "Reference" "#PWR083"
+		(property "Reference" "#PWR087"
 			(at 113.03 167.64 0)
 			(hide yes)
@@
 			(project "LSR_FLCM0001_A03"
 				(path "/1e96c69b-f36f-4762-8445-55c423e1825d/3509533b-a3f9-46e2-8669-77eba5e31bfb"
-					(reference "#PWR083")
+					(reference "#PWR087")
 					(unit 1)
 				)
@@
 		(dnp no)
 		(fields_autoplaced yes)
-		(property "Reference" "R26"
+		(property "Reference" "R30"
 			(at 68.6001 97.79 90)
 			(show_name no)
@@
 			(project "LSR_FLCM0001_A03"
 				(path "/1e96c69b-f36f-4762-8445-55c423e1825d/3509533b-a3f9-46e2-8669-77eba5e31bfb"
-					(reference "R26")
+					(reference "R30")
 					(unit 1)
 					(variant
@@
 		(dnp no)
 		(fields_autoplaced yes)
-		(property "Reference" "D6"
+		(property "Reference" "D10"
 			(at 115.57 149.7964 90)
 			(show_name no)
@@
 			(project "LSR_FLCM0001_A03"
 				(path "/1e96c69b-f36f-4762-8445-55c423e1825d/3509533b-a3f9-46e2-8669-77eba5e31bfb"
-					(reference "D6")
+					(reference "D10")
 					(unit 1)
 					(variant
@@
 		(dnp no)
 		(fields_autoplaced yes)
-		(property "Reference" "R27"
+		(property "Reference" "R31"
 			(at 69.85 50.8 90)
 			(show_name no)
@@
 			(project "LSR_FLCM0001_A03"
 				(path "/1e96c69b-f36f-4762-8445-55c423e1825d/3509533b-a3f9-46e2-8669-77eba5e31bfb"
-					(reference "R27")
+					(reference "R31")
 					(unit 1)
 					(variant
@@
 		(dnp no)
 		(fields_autoplaced yes)
-		(property "Reference" "#PWR076"
+		(property "Reference" "#PWR080"
 			(at 64.77 111.76 0)
 			(hide yes)
@@
 			(project "LSR_FLCM0001_A03"
 				(path "/1e96c69b-f36f-4762-8445-55c423e1825d/3509533b-a3f9-46e2-8669-77eba5e31bfb"
-					(reference "#PWR076")
+					(reference "#PWR080")
 					(unit 1)
 				)
@@
 		(in_pos_files yes)
 		(dnp no)
-		(property "Reference" "R32"
+		(property "Reference" "R36"
 			(at 109.22 60.9599 0)
 			(show_name no)
@@
 			(project "LSR_FLCM0001_A03"
 				(path "/1e96c69b-f36f-4762-8445-55c423e1825d/3509533b-a3f9-46e2-8669-77eba5e31bfb"
-					(reference "R32")
+					(reference "R36")
 					(unit 1)
 					(variant
@@
 		(dnp no)
 		(fields_autoplaced yes)
-		(property "Reference" "D5"
+		(property "Reference" "D9"
 			(at 115.57 107.8864 90)
 			(show_name no)
@@
 			(project "LSR_FLCM0001_A03"
 				(path "/1e96c69b-f36f-4762-8445-55c423e1825d/3509533b-a3f9-46e2-8669-77eba5e31bfb"
-					(reference "D5")
+					(reference "D9")
 					(unit 1)
 					(variant
@@
 		(dnp no)
 		(fields_autoplaced yes)
-		(property "Reference" "R25"
+		(property "Reference" "R29"
 			(at 68.58 139.7 90)
 			(show_name no)
@@
 			(project "LSR_FLCM0001_A03"
 				(path "/1e96c69b-f36f-4762-8445-55c423e1825d/3509533b-a3f9-46e2-8669-77eba5e31bfb"
-					(reference "R25")
+					(reference "R29")
 					(unit 1)
 					(variant
@@
 		(dnp no)
 		(fields_autoplaced yes)
-		(property "Reference" "#PWR078"
+		(property "Reference" "#PWR082"
 			(at 66.04 64.77 0)
 			(hide yes)
@@
 			(project "LSR_FLCM0001_A03"
 				(path "/1e96c69b-f36f-4762-8445-55c423e1825d/3509533b-a3f9-46e2-8669-77eba5e31bfb"
-					(reference "#PWR078")
+					(reference "#PWR082")
 					(unit 1)
 				)
@@
 		(dnp no)
 		(fields_autoplaced yes)
-		(property "Reference" "#PWR081"
+		(property "Reference" "#PWR085"
 			(at 106.68 78.74 0)
 			(hide yes)
@@
 			(project "LSR_FLCM0001_A03"
 				(path "/1e96c69b-f36f-4762-8445-55c423e1825d/3509533b-a3f9-46e2-8669-77eba5e31bfb"
-					(reference "#PWR081")
+					(reference "#PWR085")
 					(unit 1)
 				)
@@
 		(dnp no)
 		(fields_autoplaced yes)
-		(property "Reference" "#PWR084"
+		(property "Reference" "#PWR088"
 			(at 114.3 78.74 0)
 			(hide yes)
@@
 			(project "LSR_FLCM0001_A03"
 				(path "/1e96c69b-f36f-4762-8445-55c423e1825d/3509533b-a3f9-46e2-8669-77eba5e31bfb"
-					(reference "#PWR084")
+					(reference "#PWR088")
 					(unit 1)
 				)
@@
 		(dnp no)
 		(fields_autoplaced yes)
-		(property "Reference" "#PWR077"
+		(property "Reference" "#PWR081"
 			(at 64.77 153.67 0)
 			(hide yes)
@@
 			(project "LSR_FLCM0001_A03"
 				(path "/1e96c69b-f36f-4762-8445-55c423e1825d/3509533b-a3f9-46e2-8669-77eba5e31bfb"
-					(reference "#PWR077")
+					(reference "#PWR081")
 					(unit 1)
 				)
