File: LSR_FLCM0001_A03.kicad_pcb (KiCad board)
At the start: 6 copper layers, 30 x 60 mm, 138 parts, among them IC1 FM25L04B-DG, J1 USB_C_Receptacle_USB2.0_16P, J10 SMA_Edge, J2 Conn_01x02_Pin, J3 Conn_01x02_Pin, J4 Conn_ARM_SWD_TagConnect_TC203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, J5 Micro_SD_Card_Det2, J6 2125280200, J7 1771114, J8 Header 4, J9 SMA_Edge, Q1 AON7296, Q2 AON7296, Q3 AON7296, U1 USBLC6-2SC6, U10 BMP390, U11 MAX-M10S, U12 E22-900MM22S, U2 STM32H742VGH6, U3 W25Q128JVP, U4 TPS62130A, U5 TPS2121RUXR, U6 LSM6DSM, U7 LSM6DS320, U8 LIS2MDL, U9 BMP390, Y1 ABM3B-24.000MHZ

Commit message: Changed some of the silkscreen, and added some LEDs attached to some gpio
Parts:
- removed the TP16 at (152.8, 118.0)
- added D1: Yellow, PCM_SparkFun-LED:LED_0603_1608Metric_Yellow, B.Cu at (138.5, 119.4)
- added D2: Yellow, PCM_SparkFun-LED:LED_0603_1608Metric_Yellow, B.Cu at (141.9, 119.4)
- added D3: Red, PCM_SparkFun-LED:LED_0603_1608Metric_Red, B.Cu at (140.2, 119.4)
- added D4: Red, PCM_SparkFun-LED:LED_0603_1608Metric_Red, B.Cu at (136.8, 119.4)
- added R10: R_Small_US, Resistor_SMD:R_0402_1005Metric, B.Cu at (140.2, 122.3)
- added R11: R_Small_US, Resistor_SMD:R_0402_1005Metric, B.Cu at (136.8, 122.3)
- added R8: R_Small_US, Resistor_SMD:R_0402_1005Metric, B.Cu at (138.5, 122.3)
- added R9: R_Small_US, Resistor_SMD:R_0402_1005Metric, B.Cu at (141.9, 122.3)
- J8: value Header 4 -> Conn_01x05_Pin; footprint SAMTEC THD:SAMTEC_BBL-104-X-E -> Connector_PinHeader_2.54mm:PinHeader_1x05_P2.54mm_Vertical
- moved J8 3.84 mm to (137.0, 105.0), turned to 0 degrees
- moved J2 0.50 mm to (140.7, 103.4)
- renumbered D6 to D10, D7 to D11, D8 to D12, D9 to D13, D10 to D14, D1 to D5, D2 to D6, D3 to D7, D4 to D8, D5 to D9, R8 to R12, R9 to R13, R10 to R14, R11 to R15, R12 to R16, R13 to R17, R14 to R18, R15 to R19, R16 to R20, R17 to R21, R18 to R22, R19 to R23, R20 to R24, R21 to R25, R22 to R26, R23 to R27, R24 to R28, R25 to R29, R26 to R30, R27 to R31, R28 to R32, R29 to R33, R30 to R34, R31 to R35, R32 to R36, R33 to R37, R34 to R38, R35 to R39, R36 to R40, R37 to R41, R38 to R42, TP17 to TP16, TP18 to TP17, TP19 to TP18
Connections:
- net /Sensors/Megnetometer/C1 renamed /Sensors/Magnetometer/C1
- J8 pad 1: /TIM2_CH1 -> GND
- J8 pad 2: /TIM2_CH2 -> /TIM2_CH1
- J8 pad 3: /TIM2_CH3 -> /TIM2_CH2
- J8 pad 4: /TIM2_CH4 -> /TIM2_CH3
Routing:
- net /MCU/PE14: track 0.57 -> 33.2 mm, vias 1 -> 2
- net /MCU/PD15: track 0.57 -> 32.5 mm, vias 1 -> 2
- net /MCU/PE15: track 0.57 -> 32.2 mm, vias 1 -> 2
- net /MCU/PD14: track 0.57 -> 30.8 mm, vias 1 -> 2
- net GND: track 184.1 -> 193.4 mm
- net /ADC1_INP9: track 32.6 -> 34.4 mm
- net /TIM2_CH3: track 13.5 -> 15.3 mm
- net /ADC1_INP8: track 30.0 -> 31.8 mm
- net /TIM2_CH4: track 14.9 -> 16.6 mm
- net /ADC1_INP4: track 28.9 -> 30.6 mm
- net /MCU/USB_LED: track 0.00 -> 1.60 mm
- net /MCU/Power_LED_VIN: track 0.00 -> 1.60 mm
- net /MCU/Power_LED_3V3: track 0.00 -> 1.60 mm
- net /MCU/BATT_LED: track 0.00 -> 1.60 mm
- net VIN: track 24.1 -> 22.8 mm
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Other:
- board text added: "-"
- board text added: "1"
- board text added: "4"

Commit message: Silkscreen
Parts:
- added G***: LOGO, LSR_26-27_Library_Footprint:Eclipse2_15x5.3mm, F.Cu at (149.4, 81.0)
- added G***: LOGO, LSR_25-26_Library_Footprint:LSR_5.4x1.6mm, F.Cu at (139.9, 108.8)
- added G***: LOGO, LSR_25-26_Library_Footprint:LSR_5.4x1.6mm, B.Cu at (139.6, 100.3)
- moved TP5 0.31 mm to (151.8, 86.4)
Other:
- board text added: "FLCM0001-A03"
- board text added: "Louisiana"
- board text added: "Rocketry"
- board text added: "State"
- board text added: "lsr@lsrocketry.us"

Commit message: Silkscreen
Parts:
- added G***: LOGO, LSR_26-27_Library_Footprint:Eclipse2_14x5mm, F.Cu at (149.6, 80.7)
- added G***: LOGO, LSR_25-26_Library_Footprint:LSR_5.4x1.6mm, F.Cu at (143.1, 99.9)
- moved G*** 26.6 mm to (122.9, 80.9)
- moved G*** 12.7 mm to (127.3, 107.2)
- moved TP15 2.13 mm to (138.0, 92.1)
- moved TP2 0.69 mm to (155.6, 105.8)
- moved G*** 0.43 mm to (139.3, 100.6)
- moved TP6 0.22 mm to (152.0, 87.3)
- moved TP5 0.19 mm to (152.0, 86.4)
Other:
- board text added: "Louisiana State"
